File: Breadboard/kGeigie.kicad_sch (KiCad schematic)
At the start: 12 parts

Commit message: Updated schematic and PDF
Parts:
- removed ? (x2): (no value), symbol kGeigie-rescue:R
- removed ?: (no value), symbol kGeigie-rescue:JACK_2P
Other:
- note added: "kGeigie Schematics for M5Stack Core"
- note removed: "kGeigie Schematics"
Changed lines of the file:
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@@
 (kicad_sch (version 20220929) (generator eeschema)
   (paper "A4")
-  (junction (at 96.52 135.89) (diameter 0) (color 0 0 0 0)
-  )
-  (junction (at 109.22 125.73) (diameter 0) (color 0 0 0 0)
-  )
-  (junction (at 109.22 90.17) (diameter 0) (color 0 0 0 0)
+  (title_block
+    (date "2022-10-03")
+    (rev "V1.0")
   )
   (junction (at 88.9 73.66) (diameter 0) (color 0 0 0 0)
   )
-  (junction (at 109.22 140.97) (diameter 0) (color 0 0 0 0)
-  )
   (junction (at 137.16 90.17) (diameter 0) (color 0 0 0 0)
   )
   (junction (at 93.98 99.06) (diameter 0) (color 0 0 0 0)
   )
-  (wire (pts (xy 109.22 139.7) (xy 109.22 140.97))
-    (stroke (width 0) (type default))
-  )
-  (wire (pts (xy 96.52 125.73) (xy 109.22 125.73))
-    (stroke (width 0) (type default))
-  )
   (wire (pts (xy 88.9 85.09) (xy 88.9 73.66))
     (stroke (width 0) (type default))
@@
     (stroke (width 0) (type default))
   )
-  (wire (pts (xy 109.22 140.97) (xy 109.22 143.51))
-    (stroke (width 0) (type default))
-  )
   (wire (pts (xy 157.48 54.61) (xy 157.48 58.42))
     (stroke (width 0) (type default))
   )
-  (wire (pts (xy 96.52 140.97) (xy 109.22 140.97))
-    (stroke (width 0) (type default))
-  )
   (wire (pts (xy 86.614 73.66) (xy 88.9 73.66))
     (stroke (width 0) (type default))
@@
     (stroke (width 0) (type default))
   )
-  (wire (pts (xy 96.52 132.08) (xy 96.52 135.89))
-    (stroke (width 0) (type default))
-  )
   (wire (pts (xy 93.98 95.25) (xy 93.98 99.06))
     (stroke (width 0) (type default))
@@
     (stroke (width 0) (type default))
   )
-  (wire (pts (xy 96.52 135.89) (xy 96.52 140.97))
-    (stroke (width 0) (type default))
-  )
   (wire (pts (xy 73.66 69.85) (xy 73.66 90.424))
     (stroke (width 0) (type default))
@@
     (stroke (width 0) (type default))
   )
-  (wire (pts (xy 109.22 90.17) (xy 116.84 90.17))
-    (stroke (width 0) (type default))
-  )
-  (wire (pts (xy 109.22 90.17) (xy 109.22 114.3))
-    (stroke (width 0) (type default))
-  )
   (wire (pts (xy 124.46 90.17) (xy 127 90.17))
     (stroke (width 0) (type default))
@@
     (stroke (width 0) (type default))
   )
-  (wire (pts (xy 96.52 135.89) (xy 99.06 135.89))
-    (stroke (width 0) (type default))
-  )
-  (wire (pts (xy 99.06 135.89) (xy 99.06 129.54))
-    (stroke (width 0) (type default))
-  )
   (wire (pts (xy 73.66 90.424) (xy 78.74 90.424))
     (stroke (width 0) (type default))
@@
     (stroke (width 0) (type default))
   )
-  (wire (pts (xy 99.06 129.54) (xy 96.52 129.54))
-    (stroke (width 0) (type default))
-  )
-  (wire (pts (xy 109.22 121.92) (xy 109.22 125.73))
-    (stroke (width 0) (type default))
-  )
-  (wire (pts (xy 101.6 90.17) (xy 109.22 90.17))
-    (stroke (width 0) (type default))
-  )
-  (wire (pts (xy 109.22 125.73) (xy 109.22 132.08))
+  (wire (pts (xy 101.6 90.17) (xy 116.84 90.17))
     (stroke (width 0) (type default))
   )
@@
     (effects (font (size 1.524 1.524)) (justify left bottom))
   )
-  (text "kGeigie Schematics" (at 187.96 190.5 0)
+  (text "kGeigie Schematics for M5Stack Core" (at 187.96 190.5 0)
     (effects (font (size 1.524 1.524)) (justify left bottom))
   )
@@
     )
     (property "Datasheet" "" (at 97.79 90.17 0)
-      (effects (font (size 1.27 1.27)))
-    )
-    (pin "1")
-    (pin "2")
-  )
-  (symbol (lib_id "kGeigie-rescue:R") (at 109.22 118.11 0) (unit 1)
-    (in_bom yes) (on_board yes) (dnp no)
-    (default_instance (reference "") (unit 1) (value "") (footprint ""))
-    (property "Reference" "" (at 110.998 116.9416 0)
-      (effects (font (size 1.27 1.27)) (justify left))
-    )
-    (property "Value" "" (at 110.998 119.253 0)
-      (effects (font (size 1.27 1.27)) (justify left))
-    )
-    (property "Footprint" "" (at 107.442 118.11 90)
-      (effects (font (size 1.27 1.27)))
-    )
-    (property "Datasheet" "" (at 109.22 118.11 0)
-      (effects (font (size 1.27 1.27)))
-    )
-    (pin "1")
-    (pin "2")
-  )
-  (symbol (lib_id "kGeigie-rescue:R") (at 109.22 135.89 0) (unit 1)
-    (in_bom yes) (on_board yes) (dnp no)
-    (default_instance (reference "") (unit 1) (value "") (footprint ""))
-    (property "Reference" "" (at 110.998 134.7216 0)
-      (effects (font (size 1.27 1.27)) (justify left))
-    )
-    (property "Value" "" (at 110.998 137.033 0)
-      (effects (font (size 1.27 1.27)) (justify left))
-    )
-    (property "Footprint" "" (at 107.442 135.89 90)
-      (effects (font (size 1.27 1.27)))
-    )
-    (property "Datasheet" "" (at 109.22 135.89 0)
       (effects (font (size 1.27 1.27)))
     )
@@
     (pin "1")
   )
-  (symbol (lib_id "kGeigie-rescue:GND") (at 109.22 143.51 0) (unit 1)
-    (in_bom yes) (on_board yes) (dnp no)
-    (default_instance (reference "") (unit 1) (value "") (footprint ""))
-    (property "Reference" "" (at 109.22 149.86 0)
-      (effects (font (size 1.27 1.27)) hide)
-    )
-    (property "Value" "" (at 109.347 147.9042 0)
-      (effects (font (size 1.27 1.27)))
-    )
-    (property "Footprint" "" (at 109.22 143.51 0)
-      (effects (font (size 1.27 1.27)))
-    )
-    (property "Datasheet" "" (at 109.22 143.51 0)
-      (effects (font (size 1.27 1.27)))
-    )
-    (pin "1")
-  )
   (symbol (lib_id "kGeigie-rescue:+3.3V") (at 157.48 54.61 0) (unit 1)
     (in_bom yes) (on_board yes) (dnp no)
@@
     )
     (pin "1")
-  )
-  (symbol (lib_id "kGeigie-rescue:JACK_2P") (at 85.09 129.54 0) (unit 1)
-    (in_bom yes) (on_board yes) (dnp no)
-    (default_instance (reference "") (unit 1) (value "") (footprint ""))
-    (property "Reference" "" (at 85.2424 120.015 0)
-      (effects (font (size 1.27 1.27)))
-    )
-    (property "Value" "" (at 85.2424 122.3264 0)
-      (effects (font (size 1.27 1.27)))
-    )
-    (property "Footprint" "" (at 85.09 129.54 0)
-      (effects (font (size 1.27 1.27)))
-    )
-    (property "Datasheet" "" (at 85.09 129.54 0)
-      (effects (font (size 1.27 1.27)))
-    )
-    (pin "1")
-    (pin "2")
-    (pin "3")
   )
   (symbol (lib_id "kGeigie-rescue:Screw_Terminal_1x03") (at 80.01 90.17 0) (unit 1)
@@
       (reference "#PWR2") (unit 1) (value "GND") (footprint "")
     )
-    (path "/00000000-0000-0000-0000-000058319340"
-      (reference "#PWR3") (unit 1) (value "GND") (footprint "")
-    )
     (path "/00000000-0000-0000-0000-0000583192d3"
       (reference "#PWR4") (unit 1) (value "GND") (footprint "")
@@
       (reference "J1") (unit 1) (value "IRover") (footprint "")
     )
-    (path "/00000000-0000-0000-0000-000058319dc7"
-      (reference "J2") (unit 1) (value "JACK_2P") (footprint "")
-    )
     (path "/00000000-0000-0000-0000-000058317ee8"
       (reference "Q1") (unit 1) (value "C1815") (footprint "")
@@
       (reference "R1") (unit 1) (value "4.7k") (footprint "")
     )
-    (path "/00000000-0000-0000-0000-000058317c74"
-      (reference "R2") (unit 1) (value "47k") (footprint "")
-    )
-    (path "/00000000-0000-0000-0000-000058317ca9"
-      (reference "R3") (unit 1) (value "4.7k") (footprint "")
-    )
     (path "/00000000-0000-0000-0000-000058317cd3"
